File: hardware/thin18-compact/c4d14-96x68-routed-working/eda/core/PANDA-STD-CORE-EVT/PANDA-THIN16/PANDA-STD-CORE-EVT-quilter-j501-merged.kicad_pcb (KiCad board)
At the start: 4 copper layers, 96 x 68 mm, 189 parts, among them J201 USB4500-03-0-A, J301 DF58-2P-1.2V(21), J302 SM03B-SRSS-TB NTC, J501 104031-0811 / microSD, J502 SM02B-SRSS-TB, J503 TC2030-IDC-NL / DEBUG, J802 FH12-24S-0.5SH(55), J803 FH34SRJ-6S-0.5SH(50), J804 FH34SRJ-6S-0.5SH(50), Q801 NX3008NBK,215, SW201 SKSCLCE010, SW202 SKSCLCE010, U302 RV-3028-C7, U402 TPS22916CYFPT, U403 TPS22916CYFPT, U404 TPS22916CYFPT, U405 TPS22916CYFPT, U501 ESP32-S3-WROOM-1U-N16R8, U503 QMI8658A, U601 XL9535, U801 AIP74LVC2G17GC363.TR, U802 AIP74LVC2G17GC363.TR, U803 AIP74LVC2G17GC363.TR, U901 SGM41513YTQF24G/TR, U902 SGM62125AXG/TR, U903 CW2217BAAD, U904 NS4168, U905 SGM37601YTRL20G/TR

Commit message: feat(hw): close compact 3v3 aon route
Routing:
- net BQ_INT: track 42.7 -> 0.00 mm, vias 3 -> 0
- net 3V3_AON: track 339.0 -> 332.2 mm
