File: hardware/thin18-compact/core-c1-96x68-split/eda/core/PANDA-STD-CORE-EVT/PANDA-THIN16/usb-interface.kicad_sch (KiCad schematic)
At the start: 10 parts, among them J201 USB4500-03-0-A

Commit message: feat(hw): audit split stack and verify exact-part sourcing
Parts:
- D201: LCSC (none) -> C138714
- D202: LCSC (none) -> C48260
- J201: LCSC (none) -> C5354966

Commit message: hw: apply reviewed domestic ECOs and gate incomplete Split-C1 orders
Parts:
- R529, R530: LCSC C25092 -> C324769; MPN 0402WGF220JTCE -> RC-02K22R0FT; Manufacturer UNI-ROYAL -> FH (Fenghua Advanced)

Commit message: hw: replace USB-C with MUP and clear standard board-edge DFM
Parts:
- J201: value USB4500-03-0-A -> U20405-01 USB2.0; footprint panda-layout:USB4500_08mm_MidMount_LayoutReview -> panda-standard:MUP_U20405_01_R4; LCSC C5354966 -> C20624794; MPN USB4500-03-0-A -> U20405-01; Manufacturer GCT -> MUP

Commit message: hw: replace Split-C1 VBUS TVS with polarized SGMICRO protection
Parts:
- D202: value TPD1E10B06DPYR -> SGM05HU1ALXUGY2G/TR; footprint Package_SON:Texas_DPY0002A_0.6x1mm_P0.65mm -> panda-standard:SGM05HU1AL_UTDFN_1006_2BL; symbol panda-standard:TPD1E10B06DPYR -> panda-standard:SGM05HU1ALXUGY2G_TR; LCSC C48260 -> (none); MPN TPD1E10B06DPYR -> SGM05HU1ALXUGY2G/TR; Manufacturer Texas Instruments -> SGMICRO

Commit message: hardware: close three imported Split-C1 refs and two SMT maps
Parts:
- D201: value TPD4E05U06DQAR -> LRC8804FDT1G; footprint Package_SON:USON-10_2.5x1.0mm_P0.5mm -> panda-standard:LRC8804F_DFN2510; symbol panda-standard:TPD4E05U06DQAR -> panda-standard:LRC8804FDT1G; LCSC C138714 -> C2856698; MPN TPD4E05U06DQAR -> LRC8804FDT1G; Manufacturer Texas Instruments -> LRC
- D202: LCSC (none) -> C55274065
